File: hardware/proto-switch/tbge.sch (KiCad schematic (older format))
At the start: 29 parts, among them IC402 ECMF04-4HSM10, IC404 ECMF04-4HSM10, IC406 ECMF04-4HSM10, IC408 ECMF04-4HSM10, J401 RJHSE-538x-04

Commit message: rtm proto sensor and switch
Parts:
- R401, R403, R407, R409, R413, R415, R419, R421: Farnell (none) -> 2331474; Voltage (none) -> 50
- R402, R404, R405, R408, R410, R411, R414, R416, R417, R420, R422, R423: Farnell (none) -> 2302541; Voltage (none) -> 50
- R406, R412, R418, R424: Farnell (none) -> 9239111; Voltage (none) -> 50
Changed lines of the file:
@@
 F 2 "agg:0402" H 6300 2000 50  0001 C CNN
 F 3 "" H 6300 2000 50  0001 C CNN
+F 4 "2331474" H 0   0   50  0001 C CNN "Farnell"
+F 5 "50" H 0   0   50  0001 C CNN "Voltage"
 	1    6300 2000
 	1    0    0    -1
@@
 F 2 "agg:0402" H 6300 2300 50  0001 C CNN
 F 3 "" H 6300 2300 50  0001 C CNN
+F 4 "2331474" H 0   0   50  0001 C CNN "Farnell"
+F 5 "50" H 0   0   50  0001 C CNN "Voltage"
 	1    6300 2300
 	1    0    0    -1
@@
 F 2 "agg:0402" H 1950 1950 50  0001 C CNN
 F 3 "" H 1950 1950 50  0001 C CNN
+F 4 "9239111" H 0   0   50  0001 C CNN "Farnell"
+F 5 "50" H 0   0   50  0001 C CNN "Voltage"
 	1    1950 1950
 	0    1    -1   0
@@
 F 2 "agg:0402" H 1800 1600 50  0001 C CNN
 F 3 "" H 1800 1600 50  0001 C CNN
+F 4 "2302541" H 0   0   50  0001 C CNN "Farnell"
+F 5 "50" H 0   0   50  0001 C CNN "Voltage"
 	1    1800 1600
 	-1   0    0    1
@@
 F 2 "agg:0402" H 1800 1400 50  0001 C CNN
 F 3 "" H 1800 1400 50  0001 C CNN
+F 4 "2302541" H 0   0   50  0001 C CNN "Farnell"
+F 5 "50" H 0   0   50  0001 C CNN "Voltage"
 	1    1800 1400
 	-1   0    0    1
@@
 F 2 "agg:0402" H 1950 1550 50  0001 C CNN
 F 3 "" H 1950 1550 50  0001 C CNN
+F 4 "2302541" H 0   0   50  0001 C CNN "Farnell"
+F 5 "50" H 0   0   50  0001 C CNN "Voltage"
 	1    1950 1550
 	0    1    -1   0
@@
 F 2 "agg:0402" H 6300 2600 50  0001 C CNN
 F 3 "" H 6300 2600 50  0001 C CNN
+F 4 "2331474" H 0   0   50  0001 C CNN "Farnell"
+F 5 "50" H 0   0   50  0001 C CNN "Voltage"
 	1    6300 2600
 	1    0    0    1
@@
 F 2 "agg:0402" H 6300 2900 50  0001 C CNN
 F 3 "" H 6300 2900 50  0001 C CNN
+F 4 "2331474" H 0   0   50  0001 C CNN "Farnell"
+F 5 "50" H 0   0   50  0001 C CNN "Voltage"
 	1    6300 2900
 	1    0    0    1
@@
 F 2 "agg:0402" H 1950 3150 50  0001 C CNN
 F 3 "" H 1950 3150 50  0001 C CNN
+F 4 "9239111" H 0   0   50  0001 C CNN "Farnell"
+F 5 "50" H 0   0   50  0001 C CNN "Voltage"
 	1    1950 3150
 	0    1    -1   0
@@
 F 2 "agg:0402" H 1800 2800 50  0001 C CNN
 F 3 "" H 1800 2800 50  0001 C CNN
+F 4 "2302541" H 0   0   50  0001 C CNN "Farnell"
+F 5 "50" H 0   0   50  0001 C CNN "Voltage"
 	1    1800 2800
 	-1   0    0    1
@@
 F 2 "agg:0402" H 1800 2600 50  0001 C CNN
 F 3 "" H 1800 2600 50  0001 C CNN
+F 4 "2302541" H 0   0   50  0001 C CNN "Farnell"
+F 5 "50" H 0   0   50  0001 C CNN "Voltage"
 	1    1800 2600
 	-1   0    0    1
@@
 F 2 "agg:0402" H 1950 2750 50  0001 C CNN
 F 3 "" H 1950 2750 50  0001 C CNN
+F 4 "2302541" H 0   0   50  0001 C CNN "Farnell"
+F 5 "50" H 0   0   50  0001 C CNN "Voltage"
 	1    1950 2750
 	0    1    -1   0
@@
 F 2 "agg:0402" H 6300 3200 50  0001 C CNN
 F 3 "" H 6300 3200 50  0001 C CNN
+F 4 "2331474" H 0   0   50  0001 C CNN "Farnell"
+F 5 "50" H 0   0   50  0001 C CNN "Voltage"
 	1    6300 3200
 	1    0    0    1
@@
 F 2 "agg:0402" H 6300 3500 50  0001 C CNN
 F 3 "" H 6300 3500 50  0001 C CNN
+F 4 "2331474" H 0   0   50  0001 C CNN "Farnell"
+F 5 "50" H 0   0   50  0001 C CNN "Voltage"
 	1    6300 3500
 	1    0    0    1
@@
 F 2 "agg:0402" H 1950 4350 50  0001 C CNN
 F 3 "" H 1950 4350 50  0001 C CNN
+F 4 "9239111" H 0   0   50  0001 C CNN "Farnell"
+F 5 "50" H 0   0   50  0001 C CNN "Voltage"
 	1    1950 4350
 	0    1    -1   0
@@
 F 2 "agg:0402" H 1800 4000 50  0001 C CNN
 F 3 "" H 1800 4000 50  0001 C CNN
+F 4 "2302541" H 0   0   50  0001 C CNN "Farnell"
+F 5 "50" H 0   0   50  0001 C CNN "Voltage"
 	1    1800 4000
 	-1   0    0    1
@@
 F 2 "agg:0402" H 1800 3800 50  0001 C CNN
 F 3 "" H 1800 3800 50  0001 C CNN
+F 4 "2302541" H 0   0   50  0001 C CNN "Farnell"
+F 5 "50" H 0   0   50  0001 C CNN "Voltage"
 	1    1800 3800
 	-1   0    0    1
@@
 F 2 "agg:0402" H 1950 3950 50  0001 C CNN
 F 3 "" H 1950 3950 50  0001 C CNN
+F 4 "2302541" H 0   0   50  0001 C CNN "Farnell"
+F 5 "50" H 0   0   50  0001 C CNN "Voltage"
 	1    1950 3950
 	0    1    -1   0
@@
 F 2 "agg:0402" H 6300 3800 50  0001 C CNN
 F 3 "" H 6300 3800 50  0001 C CNN
+F 4 "2331474" H 0   0   50  0001 C CNN "Farnell"
+F 5 "50" H 0   0   50  0001 C CNN "Voltage"
 	1    6300 3800
 	1    0    0    1
@@
 F 2 "agg:0402" H 6300 4100 50  0001 C CNN
 F 3 "" H 6300 4100 50  0001 C CNN
+F 4 "2331474" H 0   0   50  0001 C CNN "Farnell"
+F 5 "50" H 0   0   50  0001 C CNN "Voltage"
 	1    6300 4100
 	1    0    0    1
@@
 F 2 "agg:0402" H 1950 5550 50  0001 C CNN
 F 3 "" H 1950 5550 50  0001 C CNN
+F 4 "9239111" H 0   0   50  0001 C CNN "Farnell"
+F 5 "50" H 0   0   50  0001 C CNN "Voltage"
 	1    1950 5550
 	0    1    -1   0
@@
 F 2 "agg:0402" H 1800 5200 50  0001 C CNN
 F 3 "" H 1800 5200 50  0001 C CNN
+F 4 "2302541" H 0   0   50  0001 C CNN "Farnell"
+F 5 "50" H 0   0   50  0001 C CNN "Voltage"
 	1    1800 5200
 	-1   0    0    1
@@
 F 2 "agg:0402" H 1800 5000 50  0001 C CNN
 F 3 "" H 1800 5000 50  0001 C CNN
+F 4 "2302541" H 0   0   50  0001 C CNN "Farnell"
+F 5 "50" H 0   0   50  0001 C CNN "Voltage"
 	1    1800 5000
 	-1   0    0    1
@@
 F 2 "agg:0402" H 1950 5150 50  0001 C CNN
 F 3 "" H 1950 5150 50  0001 C CNN
+F 4 "2302541" H 0   0   50  0001 C CNN "Farnell"
+F 5 "50" H 0   0   50  0001 C CNN "Voltage"
 	1    1950 5150
 	0    1    -1   0
