File: hardware/proto-switch/proto-switch.sch (KiCad schematic (older format))
At the start: 4 parts, among them X101 M3_MOUNT, X102 M3_MOUNT, X103 M3_MOUNT, X104 M3_MOUNT

Commit message: rename to daqnet
Changed lines of the file:
@@
 encoding utf-8
 Sheet 1 5
-Title "TBGe Switch Prototype"
+Title "DAQnet Switch Prototype"
 Date "2018-11-24"
 Rev "1"
@@
 S 3200 3000 900  2650
 U 5C2ED83C
-F0 "TGBe Ports" 50
-F1 "tbge.sch" 50
+F0 "DAQnet Ports" 50
+F1 "daqnet.sch" 50
 F2 "P1_LED1" I R 4100 3450 50
 F3 "P1_LED2" I R 4100 3550 50
