File: hardware/proto-switch/daqnet.sch (KiCad schematic (older format))
At the start: 29 parts, among them IC402 ECMF04-4HSM10, IC404 ECMF04-4HSM10, IC406 ECMF04-4HSM10, IC408 ECMF04-4HSM10, J401 RJHSE-538x-04

Commit message: rename to daqnet
Parts:
- renumbered IC402 to IC?, IC404 to IC?, IC406 to IC?, IC408 to IC?, J401 to J?, R401 to R?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

Commit message: fix annotations on switch; generate BOMs
Parts:
- gave numbers to parts that had none: 29
