File: hardware/proto-switch/ethernet.sch (KiCad schematic (older format))
At the start: 42 parts, among them IC301 KSZ8081RNA, IC303 MAX5969x, J302 RJHSE-538x, T301 749013011A, Y301 25M

Commit message: rtm proto sensor and switch
Parts:
- C301, C303: Farnell (none) -> 2320923; Voltage (none) -> 16
- C302, C304, C306, C314: Farnell (none) -> 2528765; Voltage (none) -> 16
- C305: Farnell (none) -> 2320817; Voltage (none) -> 10
- C307, C308: Farnell (none) -> 431989; Voltage (none) -> 50
- R301, R302, R303, R304, R305, R306, R307: Farnell (none) -> 2302472; Voltage (none) -> 50
- R308, R310, R318: Farnell (none) -> 2331474; Voltage (none) -> 50
- R309: Farnell (none) -> 2302722; Voltage (none) -> 50
- R311: Farnell (none) -> 2302739; Voltage (none) -> 50
- R316: Farnell (none) -> 1469699; Voltage (none) -> 50
- R317: Farnell (none) -> 2302613; Voltage (none) -> 50
Changed lines of the file:
@@
 F 2 "agg:0603" H 4550 3300 50  0001 C CNN
 F 3 "" H 4550 3300 50  0001 C CNN
+F 4 "431989" H 0   0   50  0001 C CNN "Farnell"
+F 5 "50" H 0   0   50  0001 C CNN "Voltage"
 	1    4550 3300
 	0    1    1    0
@@
 F 2 "agg:0603" H 4800 3300 50  0001 C CNN
 F 3 "" H 4800 3300 50  0001 C CNN
+F 4 "431989" H 0   0   50  0001 C CNN "Farnell"
+F 5 "50" H 0   0   50  0001 C CNN "Voltage"
 	1    4800 3300
 	0    1    1    0
@@
 F 2 "agg:0402" H 4550 5300 50  0001 C CNN
 F 3 "" H 4550 5300 50  0001 C CNN
+F 4 "1469699" H 0   0   50  0001 C CNN "Farnell"
+F 5 "50" H 0   0   50  0001 C CNN "Voltage"
 	1    4550 5300
 	0    1    1    0
@@
 F 2 "agg:0402" H 4550 5750 50  0001 C CNN
 F 3 "" H 4550 5750 50  0001 C CNN
+F 4 "2302613" H 0   0   50  0001 C CNN "Farnell"
+F 5 "50" H 0   0   50  0001 C CNN "Voltage"
 	1    4550 5750
 	0    1    1    0
@@
 F 2 "agg:1206" H 4800 1500 50  0001 C CNN
 F 3 "" H 4800 1500 50  0001 C CNN
+F 4 "2320923" H 0   0   50  0001 C CNN "Farnell"
+F 5 "16" H 0   0   50  0001 C CNN "Voltage"
 	1    4800 1500
 	0    1    1    0
@@
 F 2 "agg:0402" H 5050 1500 50  0001 C CNN
 F 3 "" H 5050 1500 50  0001 C CNN
+F 4 "2528765" H 0   0   50  0001 C CNN "Farnell"
+F 5 "16" H 0   0   50  0001 C CNN "Voltage"
 	1    5050 1500
 	0    1    1    0
@@
 F 2 "agg:1206" H 4600 2000 50  0001 C CNN
 F 3 "" H 4600 2000 50  0001 C CNN
+F 4 "2320923" H 0   0   50  0001 C CNN "Farnell"
+F 5 "16" H 0   0   50  0001 C CNN "Voltage"
 	1    4600 2000
 	0    1    1    0
@@
 F 2 "agg:0402" H 4850 2000 50  0001 C CNN
 F 3 "" H 4850 2000 50  0001 C CNN
+F 4 "2528765" H 0   0   50  0001 C CNN "Farnell"
+F 5 "16" H 0   0   50  0001 C CNN "Voltage"
 	1    4850 2000
 	0    1    1    0
@@
 F 2 "agg:0603" H 5000 2200 50  0001 C CNN
 F 3 "" H 5000 2200 50  0001 C CNN
+F 4 "2320817" H 0   0   50  0001 C CNN "Farnell"
+F 5 "10" H 0   0   50  0001 C CNN "Voltage"
 	1    5000 2200
 	0    1    1    0
@@
 F 2 "agg:0402" H 5250 2200 50  0001 C CNN
 F 3 "" H 5250 2200 50  0001 C CNN
+F 4 "2528765" H 0   0   50  0001 C CNN "Farnell"
+F 5 "16" H 0   0   50  0001 C CNN "Voltage"
 	1    5250 2200
 	0    1    1    0
@@
 F 2 "agg:0402" H 6700 1850 50  0001 C CNN
 F 3 "" H 6700 1850 50  0001 C CNN
+F 4 "2302472" H 0   0   50  0001 C CNN "Farnell"
+F 5 "50" H 0   0   50  0001 C CNN "Voltage"
 	1    6700 1850
 	1    0    0    -1
@@
 F 2 "agg:0402" H 6850 1950 50  0001 C CNN
 F 3 "" H 6850 1950 50  0001 C CNN
+F 4 "2302472" H 0   0   50  0001 C CNN "Farnell"
+F 5 "50" H 0   0   50  0001 C CNN "Voltage"
 	1    6850 1950
 	1    0    0    -1
@@
 F 2 "agg:0402" H 6700 2050 50  0001 C CNN
 F 3 "" H 6700 2050 50  0001 C CNN
+F 4 "2302472" H 0   0   50  0001 C CNN "Farnell"
+F 5 "50" H 0   0   50  0001 C CNN "Voltage"
 	1    6700 2050
 	1    0    0    -1
@@
 F 2 "agg:0402" H 6850 2150 50  0001 C CNN
 F 3 "" H 6850 2150 50  0001 C CNN
+F 4 "2302472" H 0   0   50  0001 C CNN "Farnell"
+F 5 "50" H 0   0   50  0001 C CNN "Voltage"
 	1    6850 2150
 	1    0    0    -1
@@
 F 2 "agg:0402" H 7500 2600 50  0001 C CNN
 F 3 "" H 7500 2600 50  0001 C CNN
+F 4 "2331474" H 0   0   50  0001 C CNN "Farnell"
+F 5 "50" H 0   0   50  0001 C CNN "Voltage"
 	1    7500 2600
 	0    1    1    0
@@
 F 2 "agg:0402" H 6800 3050 50  0001 C CNN
 F 3 "" H 6800 3050 50  0001 C CNN
+F 4 "2302722" H 0   0   50  0001 C CNN "Farnell"
+F 5 "50" H 0   0   50  0001 C CNN "Voltage"
 	1    6800 3050
 	-1   0    0    1
@@
 F 2 "agg:0402" H 6700 3500 50  0001 C CNN
 F 3 "" H 6700 3500 50  0001 C CNN
+F 4 "2302739" H 0   0   50  0001 C CNN "Farnell"
+F 5 "50" H 0   0   50  0001 C CNN "Voltage"
 	1    6700 3500
 	0    -1   -1   0
@@
 F 2 "agg:0402" H 900 3200 50  0001 C CNN
 F 3 "" H 900 3200 50  0001 C CNN
+F 4 "2331474" H 0   0   50  0001 C CNN "Farnell"
+F 5 "50" H 0   0   50  0001 C CNN "Voltage"
 	1    900  3200
 	1    0    0    -1
@@
 F 2 "agg:0402" H 6700 2350 50  0001 C CNN
 F 3 "" H 6700 2350 50  0001 C CNN
+F 4 "2302472" H 0   0   50  0001 C CNN "Farnell"
+F 5 "50" H 0   0   50  0001 C CNN "Voltage"
 	1    6700 2350
 	1    0    0    -1
@@
 F 2 "agg:0402" H 6850 2450 50  0001 C CNN
 F 3 "" H 6850 2450 50  0001 C CNN
+F 4 "2302472" H 0   0   50  0001 C CNN "Farnell"
+F 5 "50" H 0   0   50  0001 C CNN "Voltage"
 	1    6850 2450
 	1    0    0    -1
@@
 F 2 "agg:0402" H 6700 2550 50  0001 C CNN
 F 3 "" H 6700 2550 50  0001 C CNN
+F 4 "2302472" H 0   0   50  0001 C CNN "Farnell"
+F 5 "50" H 0   0   50  0001 C CNN "Voltage"
 	1    6700 2550
 	1    0    0    -1
@@
 F 2 "agg:0402" H 950 2900 50  0001 C CNN
 F 3 "" H 950 2900 50  0001 C CNN
+F 4 "2331474" H 0   0   50  0001 C CNN "Farnell"
+F 5 "50" H 0   0   50  0001 C CNN "Voltage"
 	1    950  2900
 	1    0    0    -1
@@
 F 2 "agg:0402" H 4350 4050 50  0001 C CNN
 F 3 "" H 4350 4050 50  0001 C CNN
+F 4 "2528765" H 0   0   50  0001 C CNN "Farnell"
+F 5 "16" H 0   0   50  0001 C CNN "Voltage"
 	1    4350 4050
 	0    1    1    0

Commit message: fix annotations on switch; generate BOMs
Parts:
- C302, C304, C306, C314: Farnell 2528765 -> 2810260
Changed lines of the file:
@@
 F 2 "agg:0402" H 5050 1500 50  0001 C CNN
 F 3 "" H 5050 1500 50  0001 C CNN
-F 4 "2528765" H 0   0   50  0001 C CNN "Farnell"
+F 4 "2810260" H 0   0   50  0001 C CNN "Farnell"
 F 5 "16" H 0   0   50  0001 C CNN "Voltage"
 	1    5050 1500
@@
 F 2 "agg:0402" H 4850 2000 50  0001 C CNN
 F 3 "" H 4850 2000 50  0001 C CNN
-F 4 "2528765" H 0   0   50  0001 C CNN "Farnell"
+F 4 "2810260" H 0   0   50  0001 C CNN "Farnell"
 F 5 "16" H 0   0   50  0001 C CNN "Voltage"
 	1    4850 2000
@@
 F 2 "agg:0402" H 5250 2200 50  0001 C CNN
 F 3 "" H 5250 2200 50  0001 C CNN
-F 4 "2528765" H 0   0   50  0001 C CNN "Farnell"
+F 4 "2810260" H 0   0   50  0001 C CNN "Farnell"
 F 5 "16" H 0   0   50  0001 C CNN "Voltage"
 	1    5250 2200
@@
 F 2 "agg:0402" H 4350 4050 50  0001 C CNN
 F 3 "" H 4350 4050 50  0001 C CNN
-F 4 "2528765" H 0   0   50  0001 C CNN "Farnell"
+F 4 "2810260" H 0   0   50  0001 C CNN "Farnell"
 F 5 "16" H 0   0   50  0001 C CNN "Voltage"
 	1    4350 4050
