File: hardware/proto-switch/ice40.sch (KiCad schematic (older format))
At the start: 47 parts, among them IC201 W25Q80, IC202 iCE40HX8K-BG121, J202 UART, Y201 25M

Commit message: rtm proto sensor and switch
Parts:
- C201, C202, C203, C204, C205, C209, C210, C211, C212, C217, C219, C220, C222: Farnell (none) -> 2528765; Voltage (none) -> 16
- C206, C207, C208, C213, C214, C215, C216: Farnell (none) -> 2470416; Voltage (none) -> 50
- C218, C221, C223, C224: Farnell (none) -> 2611921; Voltage (none) -> 6.3
- IC202: DigiKey (none) -> 220-2148-ND; Digikey 220-2148-ND -> (none)
- J201: Farnell (none) -> 2856426
- J202: footprint agg:S04B-PASK-2 -> agg:SM04B-PASS
- R201, R202, R206, R207, R211: Farnell (none) -> 2302739; Voltage (none) -> 50
- R204, R205: Farnell (none) -> 9239111; Voltage (none) -> 50
- R208, R209, R210, R212, R213: Farnell (none) -> 2331474; Voltage (none) -> 50
Changed lines of the file:
@@
 F 2 "agg:0402" H 1400 2550 50  0001 C CNN
 F 3 "" H 1400 2550 50  0001 C CNN
+F 4 "2528765" H 0   0   50  0001 C CNN "Farnell"
+F 5 "16" H 0   0   50  0001 C CNN "Voltage"
 	1    1400 2550
 	0    1    1    0
@@
 F 2 "agg:0603" H 1150 2550 50  0001 C CNN
 F 3 "" H 1150 2550 50  0001 C CNN
+F 4 "2611921" H 0   0   50  0001 C CNN "Farnell"
+F 5 "6.3" H 0   0   50  0001 C CNN "Voltage"
 	1    1150 2550
 	0    1    1    0
@@
 F 2 "agg:0402" H 850 2500 50  0001 C CNN
 F 3 "" H 850 2500 50  0001 C CNN
+F 4 "9239111" H 0   0   50  0001 C CNN "Farnell"
+F 5 "50" H 0   0   50  0001 C CNN "Voltage"
 	1    850  2500
 	1    0    0    -1
@@
 F 2 "agg:0402" H 1400 2250 50  0001 C CNN
 F 3 "" H 1400 2250 50  0001 C CNN
+F 4 "2528765" H 0   0   50  0001 C CNN "Farnell"
+F 5 "16" H 0   0   50  0001 C CNN "Voltage"
 	1    1400 2250
 	0    1    1    0
@@
 F 2 "agg:0603" H 1150 2250 50  0001 C CNN
 F 3 "" H 1150 2250 50  0001 C CNN
+F 4 "2611921" H 0   0   50  0001 C CNN "Farnell"
+F 5 "6.3" H 0   0   50  0001 C CNN "Voltage"
 	1    1150 2250
 	0    1    1    0
@@
 F 2 "agg:0402" H 850 2200 50  0001 C CNN
 F 3 "" H 850 2200 50  0001 C CNN
+F 4 "9239111" H 0   0   50  0001 C CNN "Farnell"
+F 5 "50" H 0   0   50  0001 C CNN "Voltage"
 	1    850  2200
 	1    0    0    -1
@@
 F 2 "agg:0402" H 1000 3850 50  0001 C CNN
 F 3 "" H 1000 3850 50  0001 C CNN
+F 4 "2302739" H 0   0   50  0001 C CNN "Farnell"
+F 5 "50" H 0   0   50  0001 C CNN "Voltage"
 	1    1000 3850
 	0    1    1    0
@@
 F 2 "agg:0402" H 800 3850 50  0001 C CNN
 F 3 "" H 800 3850 50  0001 C CNN
+F 4 "2302739" H 0   0   50  0001 C CNN "Farnell"
+F 5 "50" H 0   0   50  0001 C CNN "Voltage"
 	1    800  3850
 	0    1    1    0
@@
 F 2 "agg:0402" H 1050 4550 50  0001 C CNN
 F 3 "" H 1050 4550 50  0001 C CNN
+F 4 "2302739" H 0   0   50  0001 C CNN "Farnell"
+F 5 "50" H 0   0   50  0001 C CNN "Voltage"
 	1    1050 4550
 	0    1    1    0
@@
 F 2 "agg:0402" H 4850 950 50  0001 C CNN
 F 3 "" H 4850 950 50  0001 C CNN
+F 4 "2528765" H 0   0   50  0001 C CNN "Farnell"
+F 5 "16" H 0   0   50  0001 C CNN "Voltage"
 	1    4850 950
 	0    1    1    0
@@
 F 2 "agg:0402" H 5850 950 50  0001 C CNN
 F 3 "" H 5850 950 50  0001 C CNN
+F 4 "2470416" H 0   0   50  0001 C CNN "Farnell"
+F 5 "50" H 0   0   50  0001 C CNN "Voltage"
 	1    5850 950
 	0    1    1    0
@@
 F 2 "agg:0402" H 5600 950 50  0001 C CNN
 F 3 "" H 5600 950 50  0001 C CNN
+F 4 "2470416" H 0   0   50  0001 C CNN "Farnell"
+F 5 "50" H 0   0   50  0001 C CNN "Voltage"
 	1    5600 950
 	0    1    1    0
@@
 F 2 "agg:0402" H 4600 950 50  0001 C CNN
 F 3 "" H 4600 950 50  0001 C CNN
+F 4 "2528765" H 0   0   50  0001 C CNN "Farnell"
+F 5 "16" H 0   0   50  0001 C CNN "Voltage"
 	1    4600 950
 	0    1    1    0
@@
 F 2 "agg:0402" H 5100 1650 50  0001 C CNN
 F 3 "" H 5100 1650 50  0001 C CNN
+F 4 "2528765" H 0   0   50  0001 C CNN "Farnell"
+F 5 "16" H 0   0   50  0001 C CNN "Voltage"
 	1    5100 1650
 	0    1    1    0
@@
 F 2 "agg:0402" H 5600 1650 50  0001 C CNN
 F 3 "" H 5600 1650 50  0001 C CNN
+F 4 "2470416" H 0   0   50  0001 C CNN "Farnell"
+F 5 "50" H 0   0   50  0001 C CNN "Voltage"
 	1    5600 1650
 	0    1    1    0
@@
 F 2 "agg:0402" H 5850 1650 50  0001 C CNN
 F 3 "" H 5850 1650 50  0001 C CNN
+F 4 "2470416" H 0   0   50  0001 C CNN "Farnell"
+F 5 "50" H 0   0   50  0001 C CNN "Voltage"
 	1    5850 1650
 	0    1    1    0
@@
 F 2 "agg:0402" H 4600 1650 50  0001 C CNN
 F 3 "" H 4600 1650 50  0001 C CNN
+F 4 "2528765" H 0   0   50  0001 C CNN "Farnell"
+F 5 "16" H 0   0   50  0001 C CNN "Voltage"
 	1    4600 1650
 	0    1    1    0
@@
 F 2 "agg:0402" H 5350 1650 50  0001 C CNN
 F 3 "" H 5350 1650 50  0001 C CNN
+F 4 "2528765" H 0   0   50  0001 C CNN "Farnell"
+F 5 "16" H 0   0   50  0001 C CNN "Voltage"
 	1    5350 1650
 	0    1    1    0
@@
 F 2 "agg:0402" H 6100 1650 50  0001 C CNN
 F 3 "" H 6100 1650 50  0001 C CNN
+F 4 "2470416" H 0   0   50  0001 C CNN "Farnell"
+F 5 "50" H 0   0   50  0001 C CNN "Voltage"
 	1    6100 1650
 	0    1    1    0
@@
 F 2 "agg:0402" H 6350 1650 50  0001 C CNN
 F 3 "" H 6350 1650 50  0001 C CNN
+F 4 "2470416" H 0   0   50  0001 C CNN "Farnell"
+F 5 "50" H 0   0   50  0001 C CNN "Voltage"
 	1    6350 1650
 	0    1    1    0
@@
 F 2 "agg:0402" H 4850 1650 50  0001 C CNN
 F 3 "" H 4850 1650 50  0001 C CNN
+F 4 "2528765" H 0   0   50  0001 C CNN "Farnell"
+F 5 "16" H 0   0   50  0001 C CNN "Voltage"
 	1    4850 1650
 	0    1    1    0
@@
 F 2 "agg:0402" H 10100 4100 50  0001 C CNN
 F 3 "" H 10100 4100 50  0001 C CNN
+F 4 "2331474" H 0   0   50  0001 C CNN "Farnell"
+F 5 "50" H 0   0   50  0001 C CNN "Voltage"
 	1    10100 4100
 	0    1    1    0
@@
 F 2 "agg:0402" H 10400 4100 50  0001 C CNN
 F 3 "" H 10400 4100 50  0001 C CNN
+F 4 "2331474" H 0   0   50  0001 C CNN "Farnell"
+F 5 "50" H 0   0   50  0001 C CNN "Voltage"
 	1    10400 4100
 	0    1    1    0
@@
 F 2 "agg:0402" H 10700 4100 50  0001 C CNN
 F 3 "" H 10700 4100 50  0001 C CNN
+F 4 "2331474" H 0   0   50  0001 C CNN "Farnell"
+F 5 "50" H 0   0   50  0001 C CNN "Voltage"
 	1    10700 4100
 	0    1    1    0
@@
 F 2 "agg:0402" H 6100 950 50  0001 C CNN
 F 3 "" H 6100 950 50  0001 C CNN
+F 4 "2470416" H 0   0   50  0001 C CNN "Farnell"
+F 5 "50" H 0   0   50  0001 C CNN "Voltage"
 	1    6100 950
 	0    1    1    0
@@
 F 2 "agg:0402" H 5100 950 50  0001 C CNN
 F 3 "" H 5100 950 50  0001 C CNN
+F 4 "2528765" H 0   0   50  0001 C CNN "Farnell"
+F 5 "16" H 0   0   50  0001 C CNN "Voltage"
 	1    5100 950
 	0    1    1    0
@@
 F 2 "agg:0402" H 5350 950 50  0001 C CNN
 F 3 "" H 5350 950 50  0001 C CNN
+F 4 "2528765" H 0   0   50  0001 C CNN "Farnell"
+F 5 "16" H 0   0   50  0001 C CNN "Voltage"
 	1    5350 950
 	0    1    1    0
@@
 F 2 "agg:0402" H 8050 2250 50  0001 C CNN
 F 3 "" H 8050 2250 50  0001 C CNN
+F 4 "2528765" H 0   0   50  0001 C CNN "Farnell"
+F 5 "16" H 0   0   50  0001 C CNN "Voltage"
 	1    8050 2250
 	0    1    1    0
@@
 F 2 "agg:0402" H 8600 900 50  0001 C CNN
 F 3 "" H 8600 900 50  0001 C CNN
+F 4 "2528765" H 0   0   50  0001 C CNN "Farnell"
+F 5 "16" H 0   0   50  0001 C CNN "Voltage"
 	1    8600 900
 	0    1    1    0
@@
 F 2 "agg:0402" H 9800 2100 50  0001 C CNN
 F 3 "" H 9800 2100 50  0001 C CNN
+F 4 "2528765" H 0   0   50  0001 C CNN "Farnell"
+F 5 "16" H 0   0   50  0001 C CNN "Voltage"
 	1    9800 2100
 	0    1    1    0
@@
 F 2 "agg:0402" H 8150 1150 50  0001 C CNN
 F 3 "" H 8150 1150 50  0001 C CNN
+F 4 "2302739" H 0   0   50  0001 C CNN "Farnell"
+F 5 "50" H 0   0   50  0001 C CNN "Voltage"
 	1    8150 1150
 	0    1    1    0
@@
 F 2 "agg:0402" H 7950 1150 50  0001 C CNN
 F 3 "" H 7950 1150 50  0001 C CNN
+F 4 "2302739" H 0   0   50  0001 C CNN "Farnell"
+F 5 "50" H 0   0   50  0001 C CNN "Voltage"
 	1    7950 1150
 	0    1    1    0
@@
 F 2 "agg:FTSH-105-01-F-D-K" H 10250 2000 50  0001 C CNN
 F 3 "" H 10250 2000 50  0001 C CNN
+F 4 "2856426" H 0   0   50  0001 C CNN "Farnell"
 	1    10250 2000
 	1    0    0    -1
@@
 F 2 "agg:Lattice-BG121" H 1900 700 50  0001 L CNN
 F 3 "http://www.latticesemi.com/view_document?document_id=49312" H 1900 600 50  0001 L CNN
-F 4 "220-2148-ND" H 1900 500 50  0001 L CNN "Digikey"
+F 4 "220-2148-ND" H 1900 500 50  0001 L CNN "DigiKey"
 	1    2750 4200
 	1    0    0    -1
@@
 F 0 "J202" H 9300 3900 50  0000 L CNN
 F 1 "UART" V 9250 3650 50  0000 C CNN
-F 2 "agg:S04B-PASK-2" H 9350 3800 50  0001 C CNN
+F 2 "agg:SM04B-PASS" H 9350 3800 50  0001 C CNN
 F 3 "" H 9350 3800 50  0001 C CNN
 	1    9350 3800
@@
 F 2 "agg:0402" H 8550 3900 50  0001 C CNN
 F 3 "" H 8550 3900 50  0001 C CNN
+F 4 "2331474" H 0   0   50  0001 C CNN "Farnell"
+F 5 "50" H 0   0   50  0001 C CNN "Voltage"
 	1    8550 3900
 	-1   0    0    1
@@
 F 2 "agg:0402" H 8700 4000 50  0001 C CNN
 F 3 "" H 8700 4000 50  0001 C CNN
+F 4 "2331474" H 0   0   50  0001 C CNN "Farnell"
+F 5 "50" H 0   0   50  0001 C CNN "Voltage"
 	1    8700 4000
 	-1   0    0    1
@@
 F 2 "agg:0603" H 4600 2300 50  0001 C CNN
 F 3 "" H 4600 2300 50  0001 C CNN
+F 4 "2611921" H 0   0   50  0001 C CNN "Farnell"
+F 5 "6.3" H 0   0   50  0001 C CNN "Voltage"
 	1    4600 2300
 	0    1    1    0
@@
 F 2 "agg:0603" H 4850 2300 50  0001 C CNN
 F 3 "" H 4850 2300 50  0001 C CNN
+F 4 "2611921" H 0   0   50  0001 C CNN "Farnell"
+F 5 "6.3" H 0   0   50  0001 C CNN "Voltage"
 	1    4850 2300
 	0    1    1    0

Commit message: fix annotations on switch; generate BOMs
Parts:
- C201, C202, C203, C204, C205, C209, C210, C211, C212, C217, C219, C220, C222: Farnell 2528765 -> 2810260
Changed lines of the file:
@@
 F 2 "agg:0402" H 1400 2550 50  0001 C CNN
 F 3 "" H 1400 2550 50  0001 C CNN
-F 4 "2528765" H 0   0   50  0001 C CNN "Farnell"
+F 4 "2810260" H 0   0   50  0001 C CNN "Farnell"
 F 5 "16" H 0   0   50  0001 C CNN "Voltage"
 	1    1400 2550
@@
 F 2 "agg:0402" H 1400 2250 50  0001 C CNN
 F 3 "" H 1400 2250 50  0001 C CNN
-F 4 "2528765" H 0   0   50  0001 C CNN "Farnell"
+F 4 "2810260" H 0   0   50  0001 C CNN "Farnell"
 F 5 "16" H 0   0   50  0001 C CNN "Voltage"
 	1    1400 2250
@@
 F 2 "agg:0402" H 4850 950 50  0001 C CNN
 F 3 "" H 4850 950 50  0001 C CNN
-F 4 "2528765" H 0   0   50  0001 C CNN "Farnell"
+F 4 "2810260" H 0   0   50  0001 C CNN "Farnell"
 F 5 "16" H 0   0   50  0001 C CNN "Voltage"
 	1    4850 950
@@
 F 2 "agg:0402" H 4600 950 50  0001 C CNN
 F 3 "" H 4600 950 50  0001 C CNN
-F 4 "2528765" H 0   0   50  0001 C CNN "Farnell"
+F 4 "2810260" H 0   0   50  0001 C CNN "Farnell"
 F 5 "16" H 0   0   50  0001 C CNN "Voltage"
 	1    4600 950
@@
 F 2 "agg:0402" H 5100 1650 50  0001 C CNN
 F 3 "" H 5100 1650 50  0001 C CNN
-F 4 "2528765" H 0   0   50  0001 C CNN "Farnell"
+F 4 "2810260" H 0   0   50  0001 C CNN "Farnell"
 F 5 "16" H 0   0   50  0001 C CNN "Voltage"
 	1    5100 1650
@@
 F 2 "agg:0402" H 4600 1650 50  0001 C CNN
 F 3 "" H 4600 1650 50  0001 C CNN
-F 4 "2528765" H 0   0   50  0001 C CNN "Farnell"
+F 4 "2810260" H 0   0   50  0001 C CNN "Farnell"
 F 5 "16" H 0   0   50  0001 C CNN "Voltage"
 	1    4600 1650
@@
 F 2 "agg:0402" H 5350 1650 50  0001 C CNN
 F 3 "" H 5350 1650 50  0001 C CNN
-F 4 "2528765" H 0   0   50  0001 C CNN "Farnell"
+F 4 "2810260" H 0   0   50  0001 C CNN "Farnell"
 F 5 "16" H 0   0   50  0001 C CNN "Voltage"
 	1    5350 1650
@@
 F 2 "agg:0402" H 4850 1650 50  0001 C CNN
 F 3 "" H 4850 1650 50  0001 C CNN
-F 4 "2528765" H 0   0   50  0001 C CNN "Farnell"
+F 4 "2810260" H 0   0   50  0001 C CNN "Farnell"
 F 5 "16" H 0   0   50  0001 C CNN "Voltage"
 	1    4850 1650
@@
 F 2 "agg:0402" H 5100 950 50  0001 C CNN
 F 3 "" H 5100 950 50  0001 C CNN
-F 4 "2528765" H 0   0   50  0001 C CNN "Farnell"
+F 4 "2810260" H 0   0   50  0001 C CNN "Farnell"
 F 5 "16" H 0   0   50  0001 C CNN "Voltage"
 	1    5100 950
@@
 F 2 "agg:0402" H 5350 950 50  0001 C CNN
 F 3 "" H 5350 950 50  0001 C CNN
-F 4 "2528765" H 0   0   50  0001 C CNN "Farnell"
+F 4 "2810260" H 0   0   50  0001 C CNN "Farnell"
 F 5 "16" H 0   0   50  0001 C CNN "Voltage"
 	1    5350 950
@@
 F 2 "agg:0402" H 8050 2250 50  0001 C CNN
 F 3 "" H 8050 2250 50  0001 C CNN
-F 4 "2528765" H 0   0   50  0001 C CNN "Farnell"
+F 4 "2810260" H 0   0   50  0001 C CNN "Farnell"
 F 5 "16" H 0   0   50  0001 C CNN "Voltage"
 	1    8050 2250
@@
 F 2 "agg:0402" H 8600 900 50  0001 C CNN
 F 3 "" H 8600 900 50  0001 C CNN
-F 4 "2528765" H 0   0   50  0001 C CNN "Farnell"
+F 4 "2810260" H 0   0   50  0001 C CNN "Farnell"
 F 5 "16" H 0   0   50  0001 C CNN "Voltage"
 	1    8600 900
@@
 F 2 "agg:0402" H 9800 2100 50  0001 C CNN
 F 3 "" H 9800 2100 50  0001 C CNN
-F 4 "2528765" H 0   0   50  0001 C CNN "Farnell"
+F 4 "2810260" H 0   0   50  0001 C CNN "Farnell"
 F 5 "16" H 0   0   50  0001 C CNN "Voltage"
 	1    9800 2100
