File: hardware/proto-switch/power.sch (KiCad schematic (older format))
At the start: 18 parts, among them IC501 TEC 2-4810, IC502 MCP1700, IC503 TEC 2-4815, J501 GND

Commit message: rtm proto sensor and switch
Parts:
- C501: Farnell (none) -> 2611921; Voltage (none) -> 6.3
- C502, C505: Farnell (none) -> 2469398; Voltage (none) -> 25
- C503: Farnell (none) -> 2528765; Voltage (none) -> 16
- C504: Farnell (none) -> 1458896; Voltage (none) -> 10
- R501, R502, R503: Farnell (none) -> 2331474; Voltage (none) -> 50
Changed lines of the file:
@@
 F 2 "agg:0402" H 6000 4250 50  0001 C CNN
 F 3 "" H 6000 4250 50  0001 C CNN
+F 4 "1458896" H 0   0   50  0001 C CNN "Farnell"
+F 5 "10" H 0   0   50  0001 C CNN "Voltage"
 	1    6000 4250
 	0    1    1    0
@@
 F 2 "agg:0402" H 4850 4200 50  0001 C CNN
 F 3 "" H 4850 4200 50  0001 C CNN
+F 4 "2528765" H 0   0   50  0001 C CNN "Farnell"
+F 5 "16" H 0   0   50  0001 C CNN "Voltage"
 	1    4850 4200
 	0    1    1    0
@@
 F 2 "agg:0603" H 4300 3150 50  0001 C CNN
 F 3 "" H 4300 3150 50  0001 C CNN
+F 4 "2611921" H 0   0   50  0001 C CNN "Farnell"
+F 5 "6.3" H 0   0   50  0001 C CNN "Voltage"
 	1    4300 3150
 	0    1    1    0
@@
 F 2 "agg:0402" H 2000 3350 50  0001 C CNN
 F 3 "" H 2000 3350 50  0001 C CNN
+F 4 "2331474" H 0   0   50  0001 C CNN "Farnell"
+F 5 "50" H 0   0   50  0001 C CNN "Voltage"
 	1    2000 3350
 	1    0    0    -1
@@
 F 2 "agg:0402" H 2000 4300 50  0001 C CNN
 F 3 "" H 2000 4300 50  0001 C CNN
+F 4 "2331474" H 0   0   50  0001 C CNN "Farnell"
+F 5 "50" H 0   0   50  0001 C CNN "Voltage"
 	1    2000 4300
 	1    0    0    -1
@@
 F 2 "agg:0603" H 4300 4100 50  0001 C CNN
 F 3 "" H 4300 4100 50  0001 C CNN
+F 4 "2469398" H 0   0   50  0001 C CNN "Farnell"
+F 5 "25" H 0   0   50  0001 C CNN "Voltage"
 	1    4300 4100
 	0    1    1    0
@@
 F 2 "agg:0603" H 4550 4100 50  0001 C CNN
 F 3 "" H 4550 4100 50  0001 C CNN
+F 4 "2469398" H 0   0   50  0001 C CNN "Farnell"
+F 5 "25" H 0   0   50  0001 C CNN "Voltage"
 	1    4550 4100
 	0    1    1    0
@@
 F 2 "agg:0402" H 4650 3300 50  0001 C CNN
 F 3 "" H 4650 3300 50  0001 C CNN
+F 4 "2331474" H 0   0   50  0001 C CNN "Farnell"
+F 5 "50" H 0   0   50  0001 C CNN "Voltage"
 	1    4650 3300
 	0    1    1    0

Commit message: fix annotations on switch; generate BOMs
Parts:
- C503: Farnell 2528765 -> 2810260
Changed lines of the file:
@@
 F 2 "agg:0402" H 4850 4200 50  0001 C CNN
 F 3 "" H 4850 4200 50  0001 C CNN
-F 4 "2528765" H 0   0   50  0001 C CNN "Farnell"
+F 4 "2810260" H 0   0   50  0001 C CNN "Farnell"
 F 5 "16" H 0   0   50  0001 C CNN "Voltage"
 	1    4850 4200
