File: hardware/proto-switch/proto-switch.kicad_pcb (KiCad board)
At the start: 4 copper layers, 112 x 42 mm, 140 parts, among them IC201 W25Q80, IC202 iCE40HX8K-BG121, IC301 KSZ8081RNA, IC303 MAX5969x, IC402 ECMF04-4HSM10, IC404 ECMF04-4HSM10, IC406 ECMF04-4HSM10, IC408 ECMF04-4HSM10, IC501 TEC 2-4810, IC502 MCP1700, IC503 TEC 2-4815, J202 UART, J302 RJHSE-538x, J401 RJHSE-538x-04, J501 GND, T301 749013011A, X101 M3_MOUNT, X102 M3_MOUNT, X103 M3_MOUNT, X104 M3_MOUNT, Y201 25M, Y301 25M

Commit message: fix annotations on switch; generate BOMs
Parts:
- renumbered IC402 to IC401, IC404 to IC402, IC406 to IC403, IC408 to IC404, R402 to R401, R405 to R402, R408 to R403, R411 to R404, R414 to R405, R417 to R406, R420 to R407, R423 to R408, R404 to R409, R406 to R410, R410 to R411, R416 to R413, R418 to R414, R422 to R415, R424 to R416, R401 to R417, R403 to R418, R407 to R419, R409 to R420, R413 to R421, R415 to R422, R419 to R423, R421 to R424
Connections:
- net /TGBe Ports/ETD1+ renamed /DAQnet Ports/ETD1+
- net /TGBe Ports/ETD1- renamed /DAQnet Ports/ETD1-
- net /TGBe Ports/ETD2+ renamed /DAQnet Ports/ETD2+
- net /TGBe Ports/ETD2- renamed /DAQnet Ports/ETD2-
- net /TGBe Ports/ETD3+ renamed /DAQnet Ports/ETD3+
- net /TGBe Ports/ETD3- renamed /DAQnet Ports/ETD3-
- net /TGBe Ports/ETD4+ renamed /DAQnet Ports/ETD4+
- net /TGBe Ports/ETD4- renamed /DAQnet Ports/ETD4-
- net /TGBe Ports/P1_LED1 renamed /DAQnet Ports/P1_LED1
- net /TGBe Ports/P1_LED2 renamed /DAQnet Ports/P1_LED2
- net /TGBe Ports/P2_LED1 renamed /DAQnet Ports/P2_LED1
- net /TGBe Ports/P2_LED2 renamed /DAQnet Ports/P2_LED2
- net /TGBe Ports/P3_LED1 renamed /DAQnet Ports/P3_LED1
- net /TGBe Ports/P3_LED2 renamed /DAQnet Ports/P3_LED2
- net /TGBe Ports/P4_LED1 renamed /DAQnet Ports/P4_LED1
- net /TGBe Ports/P4_LED2 renamed /DAQnet Ports/P4_LED2
- net /TGBe Ports/RD1+ renamed /DAQnet Ports/RD1+
- net /TGBe Ports/RD1- renamed /DAQnet Ports/RD1-
- net /TGBe Ports/RD2+ renamed /DAQnet Ports/RD2+
- net /TGBe Ports/RD2- renamed /DAQnet Ports/RD2-
- net /TGBe Ports/RD3+ renamed /DAQnet Ports/RD3+
- net /TGBe Ports/RD3- renamed /DAQnet Ports/RD3-
- net /TGBe Ports/RD4+ renamed /DAQnet Ports/RD4+
- net /TGBe Ports/RD4- renamed /DAQnet Ports/RD4-
- net /TGBe Ports/RX1+ renamed /DAQnet Ports/RX1+
- net /TGBe Ports/RX1- renamed /DAQnet Ports/RX1-
- net /TGBe Ports/RX2+ renamed /DAQnet Ports/RX2+
- net /TGBe Ports/RX2- renamed /DAQnet Ports/RX2-
- net /TGBe Ports/RX3+ renamed /DAQnet Ports/RX3+
- net /TGBe Ports/RX3- renamed /DAQnet Ports/RX3-
- net /TGBe Ports/RX4+ renamed /DAQnet Ports/RX4+
- net /TGBe Ports/RX4- renamed /DAQnet Ports/RX4-
- net /TGBe Ports/TD1+ renamed /DAQnet Ports/TD1+
- net /TGBe Ports/TD1- renamed /DAQnet Ports/TD1-
- net /TGBe Ports/TD2+ renamed /DAQnet Ports/TD2+
- net /TGBe Ports/TD2- renamed /DAQnet Ports/TD2-
- net /TGBe Ports/TD3+ renamed /DAQnet Ports/TD3+
- net /TGBe Ports/TD3- renamed /DAQnet Ports/TD3-
- net /TGBe Ports/TD4+ renamed /DAQnet Ports/TD4+
- net /TGBe Ports/TD4- renamed /DAQnet Ports/TD4-
- net /TGBe Ports/TX1+ renamed /DAQnet Ports/TX1+
- net /TGBe Ports/TX1- renamed /DAQnet Ports/TX1-
- net /TGBe Ports/TX2+ renamed /DAQnet Ports/TX2+
- net /TGBe Ports/TX2- renamed /DAQnet Ports/TX2-
- net /TGBe Ports/TX3+ renamed /DAQnet Ports/TX3+
- net /TGBe Ports/TX3- renamed /DAQnet Ports/TX3-
- net /TGBe Ports/TX4+ renamed /DAQnet Ports/TX4+
- net /TGBe Ports/TX4- renamed /DAQnet Ports/TX4-

Commit message: Fix minimum mask width...
Other:
- rule solder_mask_min_width: 0.25 -> 0.05
