File: hardware/proto-sensor/proto-sensor.sch (KiCad schematic (older format))
At the start: 74 parts, among them IC1 RJHSE-538x, IC2 MAX15062, IC3 MCP1700, IC4 iCE40HX8K-BG121, IC5 W25Q80, IC6 MAX11665AUT, IC7 ECMF04-4HSM10, J3 GND, P1 COAX, Y1 25M

Commit message: rtm proto sensor and switch
Parts:
- C1, C14, C2, C20, C21, C23, C24, C25, C26, C28, C30, C5, C7, C8, C9: Farnell (none) -> 2528765; Voltage Rating (none) -> 16
- C10, C11, C12, C27, C29, C3, C4, C6: Farnell (none) -> 2470416; Voltage Rating (none) -> 50
- C13, C19: Farnell (none) -> 2611921; Voltage Rating (none) -> 6.3
- C15: footprint agg:0402 -> agg:0603; Farnell (none) -> 2611921; Voltage Rating (none) -> 6.3
- C16: value 1µ 48V -> 0µ47 48V; Farnell (none) -> 2211183; Voltage Rating (none) -> 50
- C17: Farnell (none) -> 431989; Voltage Rating (none) -> 50
- C18, C22: Farnell (none) -> 1458896; Voltage Rating (none) -> 10
- IC4: DigiKey (none) -> 220-2148-ND; Digikey 220-2148-ND -> (none)
- J1: Farnell (none) -> 2856426
- R1, R10, R11, R3, R9: Farnell (none) -> 2331474; Voltage Rating (none) -> 50
- R12, R13, R14, R15, R16, R20, R21: Farnell (none) -> 2302739; Voltage Rating (none) -> 50
- R19, R2, R7, R8: Farnell (none) -> 9239111; Voltage Rating (none) -> 50
- R4, R5, R6: Farnell (none) -> 2302541; Voltage Rating (none) -> 50

Commit message: rename to daqnet
Parts:
- P1: Farnell 1608592 -> 1248952
Changed lines of the file:
@@
 EESchema Schematic File Version 4
+LIBS:proto-sensor-cache
 EELAYER 29 0
 EELAYER END
@@
 encoding utf-8
 Sheet 1 1
-Title "TBGe Sensor Prototype"
+Title "DAQnet Sensor Prototype"
 Date "2018-11-20"
 Rev "1"
@@
 F 2 "agg:BNC_PCB_RA_5-1634556-0" H 4600 4940 50  0001 C CNN
 F 3 "" H 4700 5050 50  0001 C CNN
-F 4 "1608592" H 4600 4870 50  0001 C CNN "Farnell"
+F 4 "1248952" H 4600 4870 50  0001 C CNN "Farnell"
 	1    4600 5150
 	-1   0    0    -1

Commit message: fix annotations on switch; generate BOMs
Parts:
- C1, C14, C2, C20, C21, C23, C24, C25, C26, C28, C30, C5, C7, C8, C9: Farnell 2528765 -> 2810260
Connections:
- no-connect marks 78 -> 79
Changed lines of the file:
@@
 F 3 "" H 1400 2550 50  0001 C CNN
 F 4 "16" H 0   0   50  0001 C CNN "Voltage Rating"
-F 5 "2528765" H 0   0   50  0001 C CNN "Farnell"
+F 5 "2810260" H 0   0   50  0001 C CNN "Farnell"
 	1    1400 2550
 	0    1    1    0
@@
 F 3 "" H 1400 2250 50  0001 C CNN
 F 4 "16" H 0   0   50  0001 C CNN "Voltage Rating"
-F 5 "2528765" H 0   0   50  0001 C CNN "Farnell"
+F 5 "2810260" H 0   0   50  0001 C CNN "Farnell"
 	1    1400 2250
 	0    1    1    0
@@
 F 3 "" H 4850 950 50  0001 C CNN
 F 4 "16" H 0   0   50  0001 C CNN "Voltage Rating"
-F 5 "2528765" H 0   0   50  0001 C CNN "Farnell"
+F 5 "2810260" H 0   0   50  0001 C CNN "Farnell"
 	1    4850 950
 	0    1    1    0
@@
 F 3 "" H 4600 950 50  0001 C CNN
 F 4 "16" H 0   0   50  0001 C CNN "Voltage Rating"
-F 5 "2528765" H 0   0   50  0001 C CNN "Farnell"
+F 5 "2810260" H 0   0   50  0001 C CNN "Farnell"
 	1    4600 950
 	0    1    1    0
@@
 F 3 "" H 5100 1650 50  0001 C CNN
 F 4 "16" H 0   0   50  0001 C CNN "Voltage Rating"
-F 5 "2528765" H 0   0   50  0001 C CNN "Farnell"
+F 5 "2810260" H 0   0   50  0001 C CNN "Farnell"
 	1    5100 1650
 	0    1    1    0
@@
 F 3 "" H 4600 1650 50  0001 C CNN
 F 4 "16" H 0   0   50  0001 C CNN "Voltage Rating"
-F 5 "2528765" H 0   0   50  0001 C CNN "Farnell"
+F 5 "2810260" H 0   0   50  0001 C CNN "Farnell"
 	1    4600 1650
 	0    1    1    0
@@
 F 3 "" H 5350 1650 50  0001 C CNN
 F 4 "16" H 0   0   50  0001 C CNN "Voltage Rating"
-F 5 "2528765" H 0   0   50  0001 C CNN "Farnell"
+F 5 "2810260" H 0   0   50  0001 C CNN "Farnell"
 	1    5350 1650
 	0    1    1    0
@@
 F 3 "" H 4850 1650 50  0001 C CNN
 F 4 "16" H 0   0   50  0001 C CNN "Voltage Rating"
-F 5 "2528765" H 0   0   50  0001 C CNN "Farnell"
+F 5 "2810260" H 0   0   50  0001 C CNN "Farnell"
 	1    4850 1650
 	0    1    1    0
@@
 F 3 "" H 7600 6050 50  0001 C CNN
 F 4 "16" H 0   0   50  0001 C CNN "Voltage Rating"
-F 5 "2528765" H 0   0   50  0001 C CNN "Farnell"
+F 5 "2810260" H 0   0   50  0001 C CNN "Farnell"
 	1    7600 6050
 	0    1    1    0
@@
 F 3 "" H 8550 4000 50  0001 C CNN
 F 4 "16" H 0   0   50  0001 C CNN "Voltage Rating"
-F 5 "2528765" H 0   0   50  0001 C CNN "Farnell"
+F 5 "2810260" H 0   0   50  0001 C CNN "Farnell"
 	1    8550 4000
 	0    1    1    0
@@
 F 3 "" H 9750 5200 50  0001 C CNN
 F 4 "16" H 0   0   50  0001 C CNN "Voltage Rating"
-F 5 "2528765" H 0   0   50  0001 C CNN "Farnell"
+F 5 "2810260" H 0   0   50  0001 C CNN "Farnell"
 	1    9750 5200
 	0    1    1    0
@@
 F 3 "" H 9200 3200 50  0001 C CNN
 F 4 "16" H 0   0   50  0001 C CNN "Voltage Rating"
-F 5 "2528765" H 0   0   50  0001 C CNN "Farnell"
+F 5 "2810260" H 0   0   50  0001 C CNN "Farnell"
 	1    9200 3200
 	0    1    1    0
@@
 F 3 "" H 5200 4700 50  0001 C CNN
 F 4 "16" H 0   0   50  0001 C CNN "Voltage Rating"
-F 5 "2528765" H 0   0   50  0001 C CNN "Farnell"
+F 5 "2810260" H 0   0   50  0001 C CNN "Farnell"
 	1    5200 4700
 	0    1    1    0
@@
 F 3 "" H 5100 950 50  0001 C CNN
 F 4 "16" H 0   0   50  0001 C CNN "Voltage Rating"
-F 5 "2528765" H 0   0   50  0001 C CNN "Farnell"
+F 5 "2810260" H 0   0   50  0001 C CNN "Farnell"
 	1    5100 950
 	0    1    1    0
@@
 F 3 "" H 5350 950 50  0001 C CNN
 F 4 "16" H 0   0   50  0001 C CNN "Voltage Rating"
-F 5 "2528765" H 0   0   50  0001 C CNN "Farnell"
+F 5 "2810260" H 0   0   50  0001 C CNN "Farnell"
 	1    5350 950
 	0    1    1    0
@@
 Wire Wire Line
 	7300 1150 8050 1150
+NoConn ~ 10350 1500
 $EndSCHEMATC
