File: hardware/proto-sensor/proto-sensor.kicad_pcb (KiCad board)
At the start: 4 copper layers, 20 x 70 mm, 74 parts, among them IC1 RJHSE-538x, IC2 MAX15062, IC3 MCP1700, IC4 iCE40HX8K-BG121, IC5 W25Q80, IC6 MAX11665AUT, IC7 ECMF04-4HSM10, J3 GND, P1 COAX, Y1 25M

Commit message: rtm proto sensor and switch
Parts:
- C15: footprint agg:0402 -> agg:0603
- moved C18 0.38 mm to (61.2, 72.2)
- moved C22 0.38 mm to (59.1, 72.2)
- moved C15 0.21 mm to (63.9, 72.2)
Connections:
- IC1 pad S1: (no net) -> Net-(IC1-PadS1)
- IC1 pad S2: (no net) -> Net-(IC1-PadS2)
Routing:
- net 3v3: track 66.3 -> 65.3 mm
- net Net-(C18-Pad1): track 3.02 -> 3.57 mm

Commit message: Fix minimum mask width...
Other:
- rule solder_mask_min_width: 0.25 -> 0.05
Changed lines of the file:
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@@
-(kicad_pcb (version 20171130) (host pcbnew 6.0.0-rc1-unknown-106eaaa~84~ubuntu18.04.1)
+(kicad_pcb (version 20171130) (host pcbnew 6.0.0-rc1-unknown-0769b04~84~ubuntu18.04.1)
   (general
     (thickness 1.6)
@@
   )
   (setup
-    (last_trace_width 0.4)
+    (last_trace_width 0.127)
     (user_trace_width 0.127)
     (user_trace_width 0.15)
@@
     (pad_drill 0.762)
     (pad_to_mask_clearance 0.02)
-    (solder_mask_min_width 0.25)
+    (solder_mask_min_width 0.05)
     (aux_axis_origin 0 0)
     (visible_elements FFFFFF5F)
