File: hardware/interposer/interposer.sch (KiCad schematic (older format))
At the start: 15 parts, among them IC101 AD8226ARMZ, IC102 AD8226ARMZ, J101 RJHSE-5381, J102 RJHSE-5381, P101 COAX, P102 COAX, U101 LT3010-5

Commit message: add interposer bom
Parts:
- U101: RS (none) -> 761-8591
Changed lines of the file:
@@
 F 2 "Package_SO:MSOP-8-1EP_3x3mm_P0.65mm_EP1.68x1.88mm" H 5450 1825 50  0001 C CNN
 F 3 "http://cds.linear.com/docs/en/datasheet/30105fe.pdf" H 5450 1500 50  0001 C CNN
+F 4 "761-8591" H 5450 1500 50  0001 C CNN "RS"
 	1    5450 1500
 	1    0    0    -1
